File: hardware/ATMEGA16M1.sch (KiCad schematic (older format))
At the start: 56 parts, among them J1 PWR, J2 USB, J3 RELAY, J4 RELAY, J5 RELAY, J6 GPIO, J7 AMP/D2A, J8 ADC, J9 CAN, SW1 RESET, SW2 FTDI, U1 NCP1117ST50T3G, U2 FT232RL, U3 ATMEGA16M1-A, U4 MCP2551-I/SN, U5 RELAY_VO14642AT, U6 RELAY_VO14642AT, U7 RELAY_VO14642AT, X1 16MHz

Commit message: gerbers (ver 0.2) sent for fabrication
Parts:
- J3: value RELAY -> RELAY1
- J4: value RELAY -> RELAY2
- J5: value RELAY -> RELAY3
Changed lines of the file:
@@
 Sheet 1 1
 Title "LFEF CAN Communication Board"
-Date "11 apr 2015"
+Date "20 apr 2015"
 Rev "0"
 Comp "Lafayette College"
@@
 P 10150 1150
 F 0 "J3" H 10150 1300 60  0000 C CNN
-F 1 "RELAY" V 10350 1150 60  0000 C CNN
+F 1 "RELAY1" V 10350 1150 60  0000 C CNN
 F 2 "" H 10150 1150 60  0000 C CNN
 F 3 "" H 10150 1150 60  0000 C CNN
@@
 P 10150 1550
 F 0 "J4" H 10150 1700 60  0000 C CNN
-F 1 "RELAY" V 10350 1550 60  0000 C CNN
+F 1 "RELAY2" V 10350 1550 60  0000 C CNN
 F 2 "" H 10150 1550 60  0000 C CNN
 F 3 "" H 10150 1550 60  0000 C CNN
@@
 P 10150 1950
 F 0 "J5" H 10150 2100 60  0000 C CNN
-F 1 "RELAY" V 10350 1950 60  0000 C CNN
+F 1 "RELAY3" V 10350 1950 60  0000 C CNN
 F 2 "" H 10150 1950 60  0000 C CNN
 F 3 "" H 10150 1950 60  0000 C CNN
